Commit message: Added gripper and gazebo problem fixed

File: open_manipulator_description/urdf/open_manipulator.gazebo.xacro (robot description, xacro)
@@ -1,32 +1,76 @@
 <?xml version="1.0"?>
 <robot xmlns:xacro="http://ros.org/wiki/xacro">
-  <!-- Gazebo Reference macro -->
-  <xacro:macro name="RefLink" params="ref">
-    <gazebo reference="${ref}">
-      <kp>1000000.0</kp>
-      <kd>100.0</kd>
-      <mu1>30.0</mu1>
-      <mu2>30.0</mu2>
-      <maxVel>1.0</maxVel>
-      <minDepth>0.001</minDepth>
-      <material>Gazebo/DarkGrey</material>
-    </gazebo>
-  </xacro:macro>
   <!-- World -->
   <gazebo reference="world"/>
   <!-- Link1 -->
-  <RefLink ref="link1"/>
+  <gazebo reference="link1">
+    <kp>1000000.0</kp>
+    <kd>100.0</kd>
+    <mu1>30.0</mu1>
+    <mu2>30.0</mu2>
+    <maxVel>1.0</maxVel>
+    <minDepth>0.001</minDepth>
+    <material>Gazebo/DarkGrey</material>
+  </gazebo>
   <!-- Link2 -->
-  <RefLink ref="link2"/>
+  <gazebo reference="link2">
+    <kp>1000000.0</kp>
+    <kd>100.0</kd>
+    <mu1>30.0</mu1>
+    <mu2>30.0</mu2>
+    <maxVel>1.0</maxVel>
+    <minDepth>0.001</minDepth>
+    <material>Gazebo/DarkGrey</material>
+  </gazebo>
   <!-- Link3 -->
-  <RefLink ref="link3"/>
+  <gazebo reference="link3">
+    <kp>1000000.0</kp>
+    <kd>100.0</kd>
+    <mu1>30.0</mu1>
+    <mu2>30.0</mu2>
+    <maxVel>1.0</maxVel>
+    <minDepth>0.001</minDepth>
+    <material>Gazebo/DarkGrey</material>
+  </gazebo>
   <!-- Link4 -->
-  <RefLink ref="link4"/>
+  <gazebo reference="link4">
+    <kp>1000000.0</kp>
+    <kd>100.0</kd>
+    <mu1>30.0</mu1>
+    <mu2>30.0</mu2>
+    <maxVel>1.0</maxVel>
+    <minDepth>0.001</minDepth>
+    <material>Gazebo/DarkGrey</material>
+  </gazebo>
   <!-- Link5 -->
-  <RefLink ref="link5"/>
+  <gazebo reference="link5">
+    <kp>1000000.0</kp>
+    <kd>100.0</kd>
+    <mu1>30.0</mu1>
+    <mu2>30.0</mu2>
+    <maxVel>1.0</maxVel>
+    <minDepth>0.001</minDepth>
+    <material>Gazebo/DarkGrey</material>
+  </gazebo>
   <!-- gripper_link -->
-  <RefLink ref="gripper_link"/>
+  <gazebo reference="gripper_link">
+    <kp>1000000.0</kp>
+    <kd>100.0</kd>
+    <mu1>30.0</mu1>
+    <mu2>30.0</mu2>
+    <maxVel>1.0</maxVel>
+    <minDepth>0.001</minDepth>
+    <material>Gazebo/DarkGrey</material>
+  </gazebo>
   <!-- gripper_link_sub -->
-  <RefLink ref="gripper_link_sub"/>
+  <RefLink ref="gripper_link_sub">
+    <kp>1000000.0</kp>
+    <kd>100.0</kd>
+    <mu1>30.0</mu1>
+    <mu2>30.0</mu2>
+    <maxVel>1.0</maxVel>
+    <minDepth>0.001</minDepth>
+    <material>Gazebo/DarkGrey</material>
+  </gazebo>
   <!-- end effector link -->
   <gazebo reference="end_effector_link">
@@ -36,4 +80,5 @@
   <gazebo>
     <plugin name="gazebo_ros_control" filename="libgazebo_ros_control.so">
+      <robotNamespace></robotNamespace>
       <controlPeriod>0.001</controlPeriod>
       <robotSimType>gazebo_ros_control/DefaultRobotHWSim</robotSimType>
@@ -50,43 +95,3 @@
     </plugin>
   </gazebo>
-  <!-- camera -->
-  <gazebo reference="camera_link">
-    <sensor type="camera" name="intel_realsense_r200">
-      <update_rate>30.0</update_rate>
-      <camera name="head">
-        <horizontal_fov>1.02974</horizontal_fov>
-        <image>
-          <width>1920</width>
-          <height>1080</height>
-          <format>R8G8B8</format>
-        </image>
-        <clip>
-          <near>0.02</near>
-          <far>300</far>
-        </clip>
-        <noise>
-          <type>gaussian</type>
-          <!-- Noise is sampled independently per pixel on each frame.
-               That pixel's noise value is added to each of its color
-               channels, which at that point lie in the range [0,1]. -->
-          <mean>0.0</mean>
-          <stddev>0.007</stddev>
-        </noise>
-      </camera>
-      <plugin name="camera_controller" filename="libgazebo_ros_camera.so">
-        <alwaysOn>true</alwaysOn>
-        <updateRate>0.0</updateRate>
-        <cameraName>camera/color</cameraName>
-        <imageTopicName>image_raw</imageTopicName>
-        <cameraInfoTopicName>camera_info</cameraInfoTopicName>
-        <frameName>camera_link</frameName>
-        <hackBaseline>0.07</hackBaseline>
-        <distortionK1>0.0</distortionK1>
-        <distortionK2>0.0</distortionK2>
-        <distortionK3>0.0</distortionK3>
-        <distortionT1>0.0</distortionT1>
-        <distortionT2>0.0</distortionT2>
-      </plugin>
-    </sensor>
-  </gazebo>
 </robot>

Commit message: MoveIt and Gazebo error fixed

File: open_manipulator_description/urdf/open_manipulator.gazebo.xacro (robot description, xacro)
@@ -1,4 +1,4 @@
 <?xml version="1.0"?>
-<robot xmlns:xacro="http://ros.org/wiki/xacro">
+<robot xmlns:xacro="http://www.ros.org/wiki/xacro">
   <!-- World -->
   <gazebo reference="world"/>
@@ -64,5 +64,5 @@
   </gazebo>
   <!-- gripper_link_sub -->
-  <RefLink ref="gripper_link_sub">
+  <gazebo reference="gripper_link_sub">
     <kp>1000000.0</kp>
     <kd>100.0</kd>

File: open_manipulator_description/urdf/open_manipulator.transmission.xacro (robot description, xacro)
@@ -1,39 +1,42 @@
 <?xml version="1.0"?>
-<robot xmlns:xacro="http://ros.org/wiki/xacro">
-  <!-- Transmission macro -->
-  <xacro:macro name="SimpleTransmissionPosition" params="joint n">
-    <transmission name="tran${n}">
-      <type>transmission_interface/SimpleTransmission</type>
-      <joint name="${joint}">
-        <hardwareInterface>hardware_interface/PositionJointInterface</hardwareInterface>
-      </joint>
-      <actuator name="motor${n}">
-        <mechanicalReduction>1</mechanicalReduction>
-      </actuator>
-    </transmission>
-  </xacro:macro>
-  <!-- Transmission macro -->
-  <xacro:macro name="SimpleTransmissionEffort" params="joint n">
-    <transmission name="tran${n}">
-      <type>transmission_interface/SimpleTransmission</type>
-      <joint name="${joint}">
-        <hardwareInterface>hardware_interface/EffortJointInterface</hardwareInterface>
-      </joint>
-      <actuator name="motor${n}">
-        <mechanicalReduction>1</mechanicalReduction>
-      </actuator>
-    </transmission>
-  </xacro:macro>
-  <!-- Transmission 1 -->
-  <xacro:SimpleTransmissionPosition n="1" joint="joint1" />
-  <!-- Transmission 2 -->
-  <xacro:SimpleTransmissionPosition n="2" joint="joint2" />
-  <!-- Transmission 3 -->
-  <xacro:SimpleTransmissionPosition n="3" joint="joint3" />
-  <!-- Transmission 4 -->
-  <xacro:SimpleTransmissionPosition n="4" joint="joint4" />
-  <!-- Transmission 5 -->
-  <xacro:SimpleTransmissionEffort n="5" joint="gripper" />
-  <!-- Transmission 6 -->
-  <xacro:SimpleTransmissionEffort n="6" joint="gripper_sub" />
+<robot xmlns:xacro="http://www.ros.org/wiki/xacro">
+    <xacro:macro name="insert_effort_transmission" params="name">
+        <transmission name="${name}_tran">
+            <type>transmission_interface/SimpleTransmission</type>
+            <joint name="${name}" >
+                <hardwareInterface>hardware_interface/EffortJointInterface</hardwareInterface>
+                <mechanicalReduction>1</mechanicalReduction>
+            </joint>
+            <actuator name="${name}_motor">
+                <hardwareInterface>hardware_interface/EffortJointInterface</hardwareInterface>
+                <mechanicalReduction>1</mechanicalReduction>
+            </actuator>
+        </transmission>
+    </xacro:macro>
+    <xacro:macro name="insert_position_transmission" params="name">
+        <transmission name="${name}_tran">
+            <type>transmission_interface/SimpleTransmission</type>
+            <joint name="${name}" >
+                <hardwareInterface>hardware_interface/PositionJointInterface</hardwareInterface>
+                <mechanicalReduction>1</mechanicalReduction>
+            </joint>
+            <actuator name="${name}_motor">
+                <hardwareInterface>hardware_interface/PositionJointInterface</hardwareInterface>
+                <mechanicalReduction>1</mechanicalReduction>
+            </actuator>
+        </transmission>
+    </xacro:macro>
+    <xacro:macro name="insert_velocity_transmission" params="name">
+        <transmission name="${name}_tran">
+            <type>transmission_interface/SimpleTransmission</type>
+            <joint name="${name}" >
+                <hardwareInterface>hardware_interface/VelocityJointInterface</hardwareInterface>
+                <mechanicalReduction>1</mechanicalReduction>
+            </joint>
+            <actuator name="${name}_motor">
+                <hardwareInterface>hardware_interface/VelocityJointInterface</hardwareInterface>
+                <mechanicalReduction>1</mechanicalReduction>
+            </actuator>
+        </transmission>
+    </xacro:macro>
 </robot>

File: open_manipulator_description/urdf/open_manipulator.urdf.xacro (robot description, xacro)
@@ -1,5 +1,5 @@
 <?xml version="1.0"?>
 <!-- Open_Manipulator Chain -->
-<robot name= "open_manipulator" xmlns:xacro="http://ros.org/wiki/xacro">
+<robot name= "open_manipulator" xmlns:xacro="http://www.ros.org/wiki/xacro">
   <!-- Link 1 -->
   <link name="link1">
@@ -33,4 +33,5 @@
     <limit velocity="4.8" effort="1" lower="${-pi*0.9}" upper="${pi*0.9}" />
   </joint>
+  <xacro:insert_position_transmission name="joint1" />
   <!--  Link 2 -->
   <link name="link2">
@@ -64,4 +65,5 @@
     <limit velocity="4.8" effort="1" lower="${-pi*0.57}" upper="${pi*0.5}" />
   </joint>
+  <xacro:insert_position_transmission name="joint2" />
   <!--  Link 3 -->
   <link name="link3">
@@ -95,4 +97,5 @@
     <limit velocity="4.8" effort="1" lower="${-pi*0.3}" upper="${pi*0.44}" />
   </joint>
+  <xacro:insert_position_transmission name="joint3" />
   <!--  Link 4 -->
   <link name="link4">
@@ -126,4 +129,5 @@
     <limit velocity="4.8" effort="1" lower="${-pi*0.57}" upper="${pi*0.65}" />
   </joint>
+  <xacro:insert_position_transmission name="joint4" />
   <!--  Link 5 -->
   <link name="link5">
@@ -157,4 +161,5 @@
     <limit velocity="4.8" effort="1" lower="-0.010" upper="0.019" />
   </joint>
+  <xacro:insert_position_transmission name="gripper" />
   <!--  Gripper link -->
   <link name="gripper_link">
@@ -189,4 +194,5 @@
     <mimic joint="gripper" multiplier="1"/>
   </joint>
+  <xacro:insert_position_transmission name="gripper_sub" />
   <!--  Gripper link sub -->
   <link name="gripper_link_sub">

File: open_manipulator_description/urdf/open_manipulator_robot.urdf.xacro (robot description, xacro)
@@ -1,5 +1,5 @@
 <?xml version="1.0"?>
 <!-- Open_Manipulator Chain -->
-<robot name="open_manipulator" xmlns:xacro="http://ros.org/wiki/xacro">
+<robot name="open_manipulator" xmlns:xacro="http://www.ros.org/wiki/xacro">
   <!-- Import Rviz colors -->
   <xacro:include filename="$(find open_manipulator_description)/urdf/materials.xacro" />
