Commit message: Fixed error between MoveIt and actual robot

File: open_manipulator_description/urdf/open_manipulator.urdf.xacro (robot description, xacro)
@@ -26,5 +26,5 @@
   </link>
   <!-- Joint 1 -->
-  <joint name="joint1" type="revolute">
+  <joint name="id_11" type="revolute">
     <parent link="link1"/>
     <child link="link2"/>
@@ -33,5 +33,5 @@
     <limit velocity="4.8" effort="1" lower="${-pi*0.9}" upper="${pi*0.9}" />
   </joint>
-  <xacro:insert_position_transmission name="joint1" />
+  <xacro:insert_position_transmission name="id_11" />
   <!--  Link 2 -->
   <link name="link2">
@@ -58,5 +58,5 @@
   </link>
   <!--  Joint 2 -->
-  <joint name="joint2" type="revolute">
+  <joint name="id_12" type="revolute">
     <parent link="link2"/>
     <child link="link3"/>
@@ -65,5 +65,5 @@
     <limit velocity="4.8" effort="1" lower="${-pi*0.57}" upper="${pi*0.5}" />
   </joint>
-  <xacro:insert_position_transmission name="joint2" />
+  <xacro:insert_position_transmission name="id_12" />
   <!--  Link 3 -->
   <link name="link3">
@@ -90,5 +90,5 @@
   </link>
   <!--  Joint 3 -->
-  <joint name="joint3" type="revolute">
+  <joint name="id_13" type="revolute">
     <parent link="link3"/>
     <child link="link4"/>
@@ -97,5 +97,5 @@
     <limit velocity="4.8" effort="1" lower="${-pi*0.3}" upper="${pi*0.44}" />
   </joint>
-  <xacro:insert_position_transmission name="joint3" />
+  <xacro:insert_position_transmission name="id_13" />
   <!--  Link 4 -->
   <link name="link4">
@@ -122,5 +122,5 @@
   </link>
   <!--  Joint 4 -->
-  <joint name="joint4" type="revolute">
+  <joint name="id_14" type="revolute">
     <parent link="link4"/>
     <child link="link5"/>
@@ -129,5 +129,5 @@
     <limit velocity="4.8" effort="1" lower="${-pi*0.57}" upper="${pi*0.65}" />
   </joint>
-  <xacro:insert_position_transmission name="joint4" />
+  <xacro:insert_position_transmission name="id_14" />
   <!--  Link 5 -->
   <link name="link5">
@@ -154,5 +154,5 @@
   </link>
   <!--  Gripper joint -->
-  <joint name="gripper" type="prismatic">
+  <joint name="id_15" type="prismatic">
     <parent link="link5"/>
     <child link="gripper_link"/>
@@ -161,5 +161,5 @@
     <limit velocity="4.8" effort="1" lower="-0.010" upper="0.019" />
   </joint>
-  <xacro:insert_position_transmission name="gripper" />
+  <xacro:insert_position_transmission name="id_15" />
   <!--  Gripper link -->
   <link name="gripper_link">
@@ -192,5 +192,5 @@
     <axis xyz="0 -1 0"/>
     <limit velocity="4.8" effort="1" lower="-0.010" upper="0.019" />
-    <mimic joint="gripper" multiplier="1"/>
+    <mimic joint="id_15" multiplier="1"/>
   </joint>
   <xacro:insert_position_transmission name="gripper_sub" />
@@ -241,11 +241,3 @@
     </inertial>
   </link>
-  <!-- Realsense Camera Joint Position -->
-  <joint name="camera_joint" type="fixed">
-    <axis xyz="0 1 0" />
-    <origin xyz="0.070 0.032 0.052" rpy="0 0 0"/>
-    <parent link="link5"/>
-    <child link="camera_link"/>
-  </joint>
-  <link name="camera_link"/>
 </robot>
